Commit message: Fixed settings

File: src/kuka_kr5/kr5_description/urdf/kr5_robot.urdf.xacro (robot description, xacro)
@@ -13,5 +13,5 @@
     <child link = "base_link" />
     <!-- -x 0.0 -y 0.5 -z 0.762 -->
-    <origin xyz="0.0 0.5 0.762" rpy="0.0 0.0 0.0" />
+    <origin xyz="0.0 1 0.762" rpy="0.0 0.0 0.0" />
   </joint>
 </robot>

Commit message: Enhance ball controller and paddle angle calculations; add end effector tracking functionality

File: src/kuka_kr5/kr5_description/urdf/kr5_robot.urdf.xacro (robot description, xacro)
@@ -14,4 +14,5 @@
     <!-- -x 0.0 -y 0.5 -z 0.762 -->
     <origin xyz="0.0 1 0.762" rpy="0.0 0.0 0.0" />
+    <!--<origin xyz="-1.685 0.8 0.762" rpy="0.0 0.0 0.0" />-->
   </joint>
 </robot>
